Commit message: Fix cer.lauch and cer_fake_arms.urdf

File: catkin_ws/src/cer_rviz/urdf/cer_fake_arms.urdf (robot description, URDF)
Before this commit: robot SIM_CER_ROBOT, 33 links, 32 joints
Links:
- link l_clavicle: geometry collision mesh filename=package://cer_rviz/cer/meshes/dae/sim_cer_l_clavicle_prt.dae scale=0.001 0.001 0.001
- link l_forearm: geometry collision mesh filename=package://cer_rviz/cer/meshes/dae/sim_cer_l_forearm_prt.dae scale=0.001 0.001 0.001
- link l_hand: geometry collision mesh filename=package://cer_rviz/cer/meshes/dae/sim_cer_l_hand_prt.dae scale=0.001 0.001 0.001
- link l_shoulder: geometry collision mesh filename=package://cer_rviz/cer/meshes/dae/sim_cer_l_shoulder_prt.dae scale=0.001 0.001 0.001
- link l_upperarm: geometry collision mesh filename=package://cer_rviz/cer/meshes/dae/sim_cer_l_upperarm_prt.dae scale=0.001 0.001 0.001; visual mesh filename=package://cer_rviz/cer/meshes/dae/colorful_fixed/sim_cer_l_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 scale=0.001 0.001 0.001
- link l_wrist_tripod_base: geometry collision mesh filename=package://cer_rviz/cer/meshes/dae/sim_cer_l_wrist_tripod_ba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 scale=0.001 0.001 0.001
- link l_wrist_tripod_pin_dummy: geometry collision mesh filename=package://cer_rviz/cer/meshes/dae/sim_cer_l_wrist_tripod_pi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 scale=0.001 0.001 0.001
- link l_wrist_tripod_slider_dummy: geometry collision mesh filename=package://cer_rviz/cer/meshes/dae/sim_cer_l_wrist_tripod_sl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 scale=0.001 0.001 0.001
- link mobile_base_body: geometry collision mesh filename=package://cer_rviz/cer/meshes/dae/colorful_fixed/sim_cer_mo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 scale=0.001 0.001 0.001; visual mesh filename=package://cer_rviz/cer/meshes/dae/colorful_fixed/sim_cer_mo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 scale=0.001 0.001 0.001
- link mobile_base_l_tyre: geometry collision mesh filename=package://cer_rviz/cer/meshes/dae/colorful_fixed/sim_cer_mo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 scale=0.001 0.001 0.001; visual mesh filename=package://cer_rviz/cer/meshes/dae/colorful_fixed/sim_cer_mo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 scale=0.001 0.001 0.001
- link mobile_base_r_tyre: geometry collision mesh filename=package://cer_rviz/cer/meshes/dae/colorful_fixed/sim_cer_mo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 scale=0.001 0.001 0.001; visual mesh filename=package://cer_rviz/cer/meshes/dae/colorful_fixed/sim_cer_mo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 scale=0.001 0.001 0.001
- link r_clavicle: geometry collision mesh filename=package://cer_rviz/cer/meshes/dae/sim_cer_r_clavicle_prt.dae scale=0.001 0.001 0.001
- link r_forearm: geometry collision mesh filename=package://cer_rviz/cer/meshes/dae/sim_cer_r_forearm_prt.dae scale=0.001 0.001 0.001
- link r_hand: geometry collision mesh filename=package://cer_rviz/cer/meshes/dae/sim_cer_r_hand_prt.dae scale=0.001 0.001 0.001
- link r_shoulder: geometry collision mesh filename=package://cer_rviz/cer/meshes/dae/sim_cer_r_shoulder_prt.dae scale=0.001 0.001 0.001
- link r_upperarm: geometry collision mesh filename=package://cer_rviz/cer/meshes/dae/sim_cer_r_upperarm_prt.dae scale=0.001 0.001 0.001; visual mesh filename=package://cer_rviz/cer/meshes/dae/colorful_fixed/sim_cer_r_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 scale=0.001 0.001 0.001
- link r_wrist_tripod_base: geometry collision mesh filename=package://cer_rviz/cer/meshes/dae/sim_cer_r_wrist_tripod_ba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 scale=0.001 0.001 0.001
- link r_wrist_tripod_pin_dummy: geometry collision mesh filename=package://cer_rviz/cer/meshes/dae/sim_cer_r_wrist_tripod_pi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 scale=0.001 0.001 0.001
- link r_wrist_tripod_slider_dummy: geometry collision mesh filename=package://cer_rviz/cer/meshes/dae/sim_cer_r_wrist_tripod_sl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 scale=0.001 0.001 0.001
- link torso_chest: geometry collision mesh filename=package://cer_rviz/cer/meshes/dae/colorful_fixed/sim_cer_to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 scale=0.001 0.001 0.001; visual mesh filename=package://cer_rviz/cer/meshes/dae/colorful_fixed/sim_cer_to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 scale=0.001 0.001 0.001
- link torso_tripod_pin_dummy: geometry collision mesh filename=package://cer_rviz/cer/meshes/dae/sim_cer_torso_tripod_pin_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 scale=0.001 0.001 0.001; visual mesh filename=package://cer_rviz/cer/meshes/dae/sim_cer_torso_tripod_pin_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 scale=0.001 0.001 0.001
- link torso_tripod_platform: geometry collision mesh filename=package://cer_rviz/cer/meshes/dae/sim_cer_torso_tripod_plat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 scale=0.001 0.001 0.001; visual mesh filename=package://cer_rviz/cer/meshes/dae/sim_cer_torso_tripod_plat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 scale=0.001 0.001 0.001
- link torso_tripod_slider_dummy: geometry collision mesh filename=package://cer_rviz/cer/meshes/dae/colorful_fixed/sim_cer_to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 scale=0.001 0.001 0.001; visual mesh filename=package://cer_rviz/cer/meshes/dae/colorful_fixed/sim_cer_to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 scale=0.001 0.001 0.001
