Commit message: Fix urdf

File: catkin_ws/src/cer_rviz/urdf/cer.urdf (robot description, URDF)
Before this commit: robot SIM_CER_ROBOT, 33 links, 32 joints
Links:
- link l_clavicle: geometry collision mesh filename=package://cer_rviz/cer/meshes/dae/sim_cer_l_clavicle_prt.dae scale=0.001 0.001 0.001; visual mesh filename=package://cer_rviz/cer/meshes/dae/sim_cer_l_clavicle_prt.dae scale=0.001 0.001 0.001
- link l_forearm: geometry collision mesh filename=package://cer_rviz/cer/meshes/dae/sim_cer_l_forearm_prt.dae scale=0.001 0.001 0.001; visual mesh filename=package://cer_rviz/cer/meshes/dae/sim_cer_l_forearm_prt.dae scale=0.001 0.001 0.001
- link l_hand: geometry collision mesh filename=package://cer_rviz/cer/meshes/dae/sim_cer_l_hand_prt.dae scale=0.001 0.001 0.001; visual mesh filename=package://cer_rviz/cer/meshes/dae/sim_cer_l_hand_prt.dae scale=0.001 0.001 0.001
- link l_shoulder: geometry collision mesh filename=package://cer_rviz/cer/meshes/dae/sim_cer_l_shoulder_prt.dae scale=0.001 0.001 0.001; visual mesh filename=package://cer_rviz/cer/meshes/dae/sim_cer_l_shoulder_prt.dae scale=0.001 0.001 0.001
- link l_upperarm: geometry collision mesh filename=package://cer_rviz/cer/meshes/dae/sim_cer_l_upperarm_prt.dae scale=0.001 0.001 0.001; visual mesh filename=package://cer_rviz/cer/meshes/dae/sim_cer_l_upperarm_prt.dae scale=0.001 0.001 0.001
- link l_wrist_tripod_base: geometry collision mesh filename=package://cer_rviz/cer/meshes/dae/sim_cer_l_wrist_tripod_ba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 scale=0.001 0.001 0.001; visual mesh filename=package://cer_rviz/cer/meshes/dae/sim_cer_l_wrist_tripod_ba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 scale=0.001 0.001 0.001
- link l_wrist_tripod_pin_dummy: geometry collision mesh filename=package://cer_rviz/cer/meshes/dae/sim_cer_l_wrist_tripod_pi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 scale=0.001 0.001 0.001; visual mesh filename=package://cer_rviz/cer/meshes/dae/sim_cer_l_wrist_tripod_pi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 scale=0.001 0.001 0.001
- link l_wrist_tripod_slider_dummy: geometry collision mesh filename=package://cer_rviz/cer/meshes/dae/sim_cer_l_wrist_tripod_sl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 scale=0.001 0.001 0.001; visual mesh filename=package://cer_rviz/cer/meshes/dae/sim_cer_l_wrist_tripod_sl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 scale=0.001 0.001 0.001
- link mobile_base_body: geometry collision mesh filename=package://cer_rviz/cer/meshes/dae/colorful_fixed/sim_cer_mo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 scale=0.001 0.001 0.001; visual mesh filename=package://cer_rviz/cer/meshes/dae/colorful_fixed/sim_cer_mo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 scale=0.001 0.001 0.001
- link mobile_base_l_tyre: geometry collision mesh filename=package://cer_rviz/cer/meshes/dae/colorful_fixed/sim_cer_mo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 scale=0.001 0.001 0.001; visual mesh filename=package://cer_rviz/cer/meshes/dae/colorful_fixed/sim_cer_mo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 scale=0.001 0.001 0.001
- link mobile_base_r_tyre: geometry collision mesh filename=package://cer_rviz/cer/meshes/dae/colorful_fixed/sim_cer_mo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 scale=0.001 0.001 0.001; visual mesh filename=package://cer_rviz/cer/meshes/dae/colorful_fixed/sim_cer_mo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 scale=0.001 0.001 0.001
- link r_clavicle: geometry collision mesh filename=package://cer_rviz/cer/meshes/dae/sim_cer_r_clavicle_prt.dae scale=0.001 0.001 0.001; visual mesh filename=package://cer_rviz/cer/meshes/dae/sim_cer_r_clavicle_prt.dae scale=0.001 0.001 0.001
- link r_forearm: geometry collision mesh filename=package://cer_rviz/cer/meshes/dae/sim_cer_r_forearm_prt.dae scale=0.001 0.001 0.001; visual mesh filename=package://cer_rviz/cer/meshes/dae/sim_cer_r_forearm_prt.dae scale=0.001 0.001 0.001
- link r_hand: geometry collision mesh filename=package://cer_rviz/cer/meshes/dae/sim_cer_r_hand_prt.dae scale=0.001 0.001 0.001; visual mesh filename=package://cer_rviz/cer/meshes/dae/sim_cer_r_hand_prt.dae scale=0.001 0.001 0.001
- link r_shoulder: geometry collision mesh filename=package://cer_rviz/cer/meshes/dae/sim_cer_r_shoulder_prt.dae scale=0.001 0.001 0.001; visual mesh filename=package://cer_rviz/cer/meshes/dae/sim_cer_r_shoulder_prt.dae scale=0.001 0.001 0.001
- link r_upperarm: geometry collision mesh filename=package://cer_rviz/cer/meshes/dae/sim_cer_r_upperarm_prt.dae scale=0.001 0.001 0.001; visual mesh filename=package://cer_rviz/cer/meshes/dae/sim_cer_r_upperarm_prt.dae scale=0.001 0.001 0.001
- link r_wrist_tripod_base: geometry collision mesh filename=package://cer_rviz/cer/meshes/dae/sim_cer_r_wrist_tripod_ba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 scale=0.001 0.001 0.001; visual mesh filename=package://cer_rviz/cer/meshes/dae/sim_cer_r_wrist_tripod_ba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 scale=0.001 0.001 0.001
- link r_wrist_tripod_pin_dummy: geometry collision mesh filename=package://cer_rviz/cer/meshes/dae/sim_cer_r_wrist_tripod_pi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 scale=0.001 0.001 0.001; visual mesh filename=package://cer_rviz/cer/meshes/dae/sim_cer_r_wrist_tripod_pi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 scale=0.001 0.001 0.001
- link r_wrist_tripod_slider_dummy: geometry collision mesh filename=package://cer_rviz/cer/meshes/dae/sim_cer_r_wrist_tripod_sl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 scale=0.001 0.001 0.001; visual mesh filename=package://cer_rviz/cer/meshes/dae/sim_cer_r_wrist_tripod_sl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 scale=0.001 0.001 0.001
- link torso_chest: geometry collision mesh filename=package://cer_rviz/cer/meshes/dae/colorful_fixed/sim_cer_to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 scale=0.001 0.001 0.001; visual mesh filename=package://cer_rviz/cer/meshes/dae/colorful_fixed/sim_cer_to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 scale=0.001 0.001 0.001
- link torso_tripod_pin_dummy: geometry collision mesh filename=package://cer_rviz/cer/meshes/dae/sim_cer_torso_tripod_pin_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 scale=0.001 0.001 0.001; visual mesh filename=package://cer_rviz/cer/meshes/dae/sim_cer_torso_tripod_pin_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 scale=0.001 0.001 0.001
- link torso_tripod_platform: geometry collision mesh filename=package://cer_rviz/cer/meshes/dae/sim_cer_torso_tripod_plat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 scale=0.001 0.001 0.001; visual mesh filename=package://cer_rviz/cer/meshes/dae/sim_cer_torso_tripod_plat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 scale=0.001 0.001 0.001
- link torso_tripod_slider_dummy: geometry collision mesh filename=package://cer_rviz/cer/meshes/dae/colorful_fixed/sim_cer_to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 scale=0.001 0.001 0.001; visual mesh filename=package://cer_rviz/cer/meshes/dae/colorful_fixed/sim_cer_to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 scale=0.001 0.001 0.001

Commit message: Cleanup and more
* Recover old version of the model (renamed 0.1)
* Use dae instead of stl
* Remove duplicated files
* Fix urdf (rviz works again)
* Move a few files around

File: catkin_ws/src/cer_rviz/urdf/cer.urdf (robot description, URDF)
Before this commit: robot SIM_CER_ROBOT, 33 links, 32 joints
Links:
- removed link l_hand
- removed link l_wrist_tripod_pin_dummy
- removed link l_wrist_tripod_slider_dummy
- removed link r_hand
- removed link r_wrist_tripod_pin_dummy
- removed link r_wrist_tripod_slider_dummy
- removed link torso_tripod_pin_dummy
- removed link torso_tripod_slider_dummy
- added link asus_xtion
- added link base_center
- added link gaze
- added link head, mass 2.0; collision mesh filename=package://cer_rviz/../../../cer-gazebo/cer/meshes/dae/sim_c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 scale=0.001 0.001 0.001; visual mesh filename=package://cer_rviz/../../../cer-gazebo/cer/meshes/dae/sim_c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 scale=0.001 0.001 0.001
- added link l_hand_paddle, mass 0.1; collision mesh filename=package://cer_rviz/../../../cer-gazebo/cer/meshes/dae/sim_c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 scale=0.001 0.001 0.001; visual mesh filename=package://cer_rviz/../../../cer-gazebo/cer/meshes/dae/sim_c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 scale=0.001 0.001 0.001
- added link l_hand_paddle_tip
- added link l_hand_root, mass 0.5; collision mesh filename=package://cer_rviz/../../../cer-gazebo/cer/meshes/dae/sim_c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 scale=0.001 0.001 0.001; visual mesh filename=package://cer_rviz/../../../cer-gazebo/cer/meshes/dae/sim_c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 scale=0.001 0.001 0.001
- added link l_hand_thumb, mass 0.1; collision mesh filename=package://cer_rviz/../../../cer-gazebo/cer/meshes/dae/sim_c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 scale=0.001 0.001 0.001; visual mesh filename=package://cer_rviz/../../../cer-gazebo/cer/meshes/dae/sim_c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 scale=0.001 0.001 0.001
- added link l_hand_thumb_tip
- added link l_wrist_tripod_pin_eq, mass 0.2; collision mesh filename=package://cer_rviz/../../../cer-gazebo/cer/meshes/dae/sim_c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 scale=0.001 0.001 0.001; visual mesh filename=package://cer_rviz/../../../cer-gazebo/cer/meshes/dae/sim_c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 scale=0.001 0.001 0.001
- added link l_wrist_tripod_slider_eq, mass 0.2; collision mesh filename=package://cer_rviz/../../../cer-gazebo/cer/meshes/dae/sim_c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 scale=0.001 0.001 0.001; visual mesh filename=package://cer_rviz/../../../cer-gazebo/cer/meshes/dae/sim_c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 scale=0.001 0.001 0.001
- added link left_camera
- added link neck, mass 0.5; collision mesh filename=package://cer_rviz/../../../cer-gazebo/cer/meshes/dae/sim_c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 scale=0.001 0.001 0.001; visual mesh filename=package://cer_rviz/../../../cer-gazebo/cer/meshes/dae/sim_c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 scale=0.001 0.001 0.001
- added link r_hand_paddle, mass 0.1; collision mesh filename=package://cer_rviz/../../../cer-gazebo/cer/meshes/dae/sim_c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 scale=0.001 0.001 0.001; visual mesh filename=package://cer_rviz/../../../cer-gazebo/cer/meshes/dae/sim_c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 scale=0.001 0.001 0.001
- added link r_hand_paddle_tip
- added link r_hand_root, mass 0.5; collision mesh filename=package://cer_rviz/../../../cer-gazebo/cer/meshes/dae/sim_c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 scale=0.001 0.001 0.001; visual mesh filename=package://cer_rviz/../../../cer-gazebo/cer/meshes/dae/sim_c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 scale=0.001 0.001 0.001
- added link r_hand_thumb, mass 0.1; collision mesh filename=package://cer_rviz/../../../cer-gazebo/cer/meshes/dae/sim_c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 scale=0.001 0.001 0.001; visual mesh filename=package://cer_rviz/../../../cer-gazebo/cer/meshes/dae/sim_c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 scale=0.001 0.001 0.001
- added link r_hand_thumb_tip
- added link r_wrist_tripod_pin_eq, mass 0.2; collision mesh filename=package://cer_rviz/../../../cer-gazebo/cer/meshes/dae/sim_c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 scale=0.001 0.001 0.001; visual mesh filename=package://cer_rviz/../../../cer-gazebo/cer/meshes/dae/sim_c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 scale=0.001 0.001 0.001
- added link r_wrist_tripod_slider_eq, mass 0.2; collision mesh filename=package://cer_rviz/../../../cer-gazebo/cer/meshes/dae/sim_c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 scale=0.001 0.001 0.001; visual mesh filename=package://cer_rviz/../../../cer-gazebo/cer/meshes/dae/sim_c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 scale=0.001 0.001 0.001
- added link right_camera
- added link torso_tripod_pin_eq, mass 0.25; collision mesh filename=package://cer_rviz/../../../cer-gazebo/cer/meshes/dae/sim_c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 scale=0.001 0.001 0.001; visual mesh filename=package://cer_rviz/../../../cer-gazebo/cer/meshes/dae/sim_c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 scale=0.001 0.001 0.001
- added link torso_tripod_slider_eq, mass 2.5; collision mesh filename=package://cer_rviz/../../../cer-gazebo/cer/meshes/dae/sim_c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 scale=0.001 0.001 0.001; visual mesh filename=package://cer_rviz/../../../cer-gazebo/cer/meshes/dae/sim_c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 scale=0.001 0.001 0.001
- link l_clavicle: mass 0.0793454 -> 0.2; geometry collision mesh filename=package://cer_rviz/../../../cer-gazebo/cer/meshes/dae/sim_c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 scale=0.001 0.001 0.001; visual mesh filename=package://cer_rviz/../../../cer-gazebo/cer/meshes/dae/sim_c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 scale=0.001 0.001 0.001
- link l_forearm: geometry collision mesh filename=package://cer_rviz/../../../cer-gazebo/cer/meshes/dae/sim_c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 scale=0.001 0.001 0.001; visual mesh filename=package://cer_rviz/../../../cer-gazebo/cer/meshes/dae/sim_c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 scale=0.001 0.001 0.001
- link l_shoulder: geometry collision mesh filename=package://cer_rviz/../../../cer-gazebo/cer/meshes/dae/sim_c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 scale=0.001 0.001 0.001; visual mesh filename=package://cer_rviz/../../../cer-gazebo/cer/meshes/dae/sim_c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 scale=0.001 0.001 0.001
- link l_upperarm: geometry collision mesh filename=package://cer_rviz/../../../cer-gazebo/cer/meshes/dae/sim_c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 scale=0.001 0.001 0.001; visual mesh filename=package://cer_rviz/../../../cer-gazebo/cer/meshes/dae/sim_c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 scale=0.001 0.001 0.001
- link l_wrist_tripod_base: mass 0.0795216 -> 0.2; geometry collision mesh filename=package://cer_rviz/../../../cer-gazebo/cer/meshes/dae/sim_c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 scale=0.001 0.001 0.001; visual mesh filename=package://cer_rviz/../../../cer-gazebo/cer/meshes/dae/sim_c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 scale=0.001 0.001 0.001
- link mobile_base_body: mass 4.0 -> 16.0; geometry collision mesh filename=package://cer_rviz/../../../cer-gazebo/cer/meshes/dae/sim_c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 scale=0.001 0.001 0.001; visual mesh filename=package://cer_rviz/../../../cer-gazebo/cer/meshes/dae/sim_c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 scale=0.001 0.001 0.001
- link mobile_base_l_tyre: geometry collision mesh filename=package://cer_rviz/../../../cer-gazebo/cer/meshes/dae/sim_c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 scale=0.001 0.001 0.001; visual mesh filename=package://cer_rviz/../../../cer-gazebo/cer/meshes/dae/sim_c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 scale=0.001 0.001 0.001
- link mobile_base_r_tyre: geometry collision mesh filename=package://cer_rviz/../../../cer-gazebo/cer/meshes/dae/sim_c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 scale=0.001 0.001 0.001; visual mesh filename=package://cer_rviz/../../../cer-gazebo/cer/meshes/dae/sim_c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 scale=0.001 0.001 0.001
- link r_clavicle: mass 0.0793454 -> 0.2; geometry collision mesh filename=package://cer_rviz/../../../cer-gazebo/cer/meshes/dae/sim_c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 scale=0.001 0.001 0.001; visual mesh filename=package://cer_rviz/../../../cer-gazebo/cer/meshes/dae/sim_c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 scale=0.001 0.001 0.001
- link r_forearm: geometry collision mesh filename=package://cer_rviz/../../../cer-gazebo/cer/meshes/dae/sim_c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 scale=0.001 0.001 0.001; visual mesh filename=package://cer_rviz/../../../cer-gazebo/cer/meshes/dae/sim_c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 scale=0.001 0.001 0.001
- link r_shoulder: geometry collision mesh filename=package://cer_rviz/../../../cer-gazebo/cer/meshes/dae/sim_c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 scale=0.001 0.001 0.001; visual mesh filename=package://cer_rviz/../../../cer-gazebo/cer/meshes/dae/sim_c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 scale=0.001 0.001 0.001
- link r_upperarm: geometry collision mesh filename=package://cer_rviz/../../../cer-gazebo/cer/meshes/dae/sim_c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 scale=0.001 0.001 0.001; visual mesh filename=package://cer_rviz/../../../cer-gazebo/cer/meshes/dae/sim_c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 scale=0.001 0.001 0.001
- link r_wrist_tripod_base: mass 0.0795216 -> 0.2; geometry collision mesh filename=package://cer_rviz/../../../cer-gazebo/cer/meshes/dae/sim_c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 scale=0.001 0.001 0.001; visual mesh filename=package://cer_rviz/../../../cer-gazebo/cer/meshes/dae/sim_c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 scale=0.001 0.001 0.001
- link torso_chest: geometry collision mesh filename=package://cer_rviz/../../../cer-gazebo/cer/meshes/dae/sim_c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 scale=0.001 0.001 0.001; visual mesh filename=package://cer_rviz/../../../cer-gazebo/cer/meshes/dae/sim_c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 scale=0.001 0.001 0.001
- link torso_tripod_platform: mass 0.131528 -> 0.25; geometry collision mesh filename=package://cer_rviz/../../../cer-gazebo/cer/meshes/dae/sim_c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 scale=0.001 0.001 0.001; visual mesh filename=package://cer_rviz/../../../cer-gazebo/cer/meshes/dae/sim_c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 scale=0.001 0.001 0.001
Joints:
- removed joint l_wrist_tripod_heave_dummy
- removed joint l_wrist_tripod_pitch_dummy
- removed joint l_wrist_tripod_roll_dummy
- removed joint r_wrist_tripod_heave_dummy
- removed joint r_wrist_tripod_pitch_dummy
- removed joint r_wrist_tripod_roll_dummy
- removed joint torso_tripod_heave_dummy
- removed joint torso_tripod_pitch_dummy
- removed joint torso_tripod_roll_dummy
- added joint asus_xtion_fixed_joint: type fixed, parent head, child asus_xtion, origin xyz=0.07702051 0 0.04662 rpy=0 0 0
- added joint base_center_fixed_joint: type fixed, parent mobile_base_body, child base_center, origin xyz=0 0 0.16 rpy=0 0 0
- added joint gaze_fixed_joint: type fixed, parent head, child gaze, origin xyz=0 0 0 rpy=0 0 0
- added joint l_hand_paddle_joint: type revolute, parent l_hand_root, child l_hand_paddle, origin xyz=0 -0.01361 -0.067977 rpy=0 0 0, axis -1.0 0.0 0.0, limit lower=0.0 upper=1.0471975511965976 effort=50000 velocity=50000
- added joint l_hand_paddle_tip_fixed_joint: type fixed, parent l_hand_paddle, child l_hand_paddle_tip, origin xyz=0 0 -0.084994 rpy=3.141592653589793 1.221730955967807 -1.5707963267948968
- added joint l_hand_thumb_joint: type revolute, parent l_hand_root, child l_hand_thumb, origin xyz=0 -0.020648 -0.042844 rpy=0 0 0, axis 1.0 0.0 0.0, limit lower=0.0 upper=1.2217304763960306 effort=50000 velocity=50000
- added joint l_hand_thumb_tip_fixed_joint: type fixed, parent l_hand_thumb, child l_hand_thumb_tip, origin xyz=0 -0.0513860000782 -0.0458929999125 rpy=3.141592653589793 1.2217309542643466 -1.570796326794897
- added joint l_wrist_tripod_heave_eq: type prismatic, parent l_wrist_tripod_base, child l_wrist_tripod_slider_eq, origin xyz=0 0 0.071 rpy=0 0 0, axis 0.0 0.0 -1.0, limit lower=0.0 upper=0.12 effort=50000 velocity=50000
- added joint l_wrist_tripod_pitch_eq: type revolute, parent l_wrist_tripod_pin_eq, child l_hand_root, origin xyz=0 0.001 0 rpy=0 -1.5707963267948966 0, axis 0.0 -1.0 0.0, limit lower=-0.5235987755982988 upper=0.5235987755982988 effort=50000 velocity=50000
- added joint l_wrist_tripod_roll_eq: type revolute, parent l_wrist_tripod_slider_eq, child l_wrist_tripod_pin_eq, origin xyz=0 0 -0.291 rpy=0 1.5707963267948966 0, axis 0.0 0.0 1.0, limit lower=-0.5235987755982988 upper=0.5235987755982988 effort=50000 velocity=50000
- added joint left_camera_fixed_joint: type fixed, parent head, child left_camera, origin xyz=0.06682051 0.0325 -0.06838 rpy=0 0 0
- added joint neck_pitch: type revolute, parent torso_chest, child neck, origin xyz=-0.094 0.000646677 0.37 rpy=0 0 0, axis 0.0 1.0 0.0, limit lower=-0.5235987755982988 upper=1.3962634015954636 effort=50000 velocity=50000
- added joint neck_yaw: type revolute, parent neck, child head, origin xyz=0.01167949 -0.000646677 0.15838 rpy=0 0 0, axis 0.173648 0.0 0.984808, limit lower=-1.3962634015954636 upper=1.3962634015954636 effort=50000 velocity=50000
- added joint r_hand_paddle_joint: type revolute, parent r_hand_root, child r_hand_paddle, origin xyz=0 0.01161 -0.067977 rpy=0 0 0, axis 1.0 0.0 0.0, limit lower=0.0 upper=1.0471975511965976 effort=50000 velocity=50000
- added joint r_hand_paddle_tip_fixed_joint: type fixed, parent r_hand_paddle, child r_hand_paddle_tip, origin xyz=0 0 -0.084994 rpy=0 1.221730955967806 1.5707963267948957
- added joint r_hand_thumb_joint: type revolute, parent r_hand_root, child r_hand_thumb, origin xyz=0 0.018648 -0.042844 rpy=0 0 0, axis -1.0 0.0 0.0, limit lower=0.0 upper=1.2217304763960306 effort=50000 velocity=50000
- added joint r_hand_thumb_tip_fixed_joint: type fixed, parent r_hand_thumb, child r_hand_thumb_tip, origin xyz=0 0.051386 -0.045893 rpy=0 1.221730955967806 1.5707963267948957
- added joint r_wrist_tripod_heave_eq: type prismatic, parent r_wrist_tripod_base, child r_wrist_tripod_slider_eq, origin xyz=0 0 0.071 rpy=0 0 0, axis 0.0 0.0 -1.0, limit lower=0.0 upper=0.12 effort=50000 velocity=50000
- added joint r_wrist_tripod_pitch_eq: type revolute, parent r_wrist_tripod_pin_eq, child r_hand_root, origin xyz=0.001 0 0 rpy=3.141592653589793 0 1.5707963267948966, axis 0.0 -1.0 0.0, limit lower=-0.5235987755982988 upper=0.5235987755982988 effort=50000 velocity=50000
- added joint r_wrist_tripod_roll_eq: type revolute, parent r_wrist_tripod_slider_eq, child r_wrist_tripod_pin_eq, origin xyz=0 0 -0.291 rpy=3.141592653589793 0 1.5707963267948966, axis 0.0 -1.0 0.0, limit lower=-0.5235987755982988 upper=0.5235987755982988 effort=50000 velocity=50000
- added joint right_camera_fixed_joint: type fixed, parent head, child right_camera, origin xyz=0.06682051 -0.0325 -0.06838 rpy=0 0 0
- added joint torso_tripod_heave_eq: type prismatic, parent mobile_base_body, child torso_tripod_slider_eq, origin xyz=0.074 0 0.231 rpy=0 0 0, axis 0.0 0.0 1.0, limit lower=-0.05 upper=0.15 effort=50000 velocity=50000
- added joint torso_tripod_pitch_eq: type revolute, parent torso_tripod_pin_eq, child torso_tripod_platform, origin xyz=0 0 0 rpy=3.141592653589793 0 0, axis 0.0 1.0 0.0, limit lower=-0.5235987755982988 upper=0.5235987755982988 effort=50000 velocity=50000
- added joint torso_tripod_roll_eq: type revolute, parent torso_tripod_slider_eq, child torso_tripod_pin_eq, origin xyz=0 0 0.399 rpy=3.141592653589793 0 0, axis 1.0 0.0 0.0, limit lower=-0.5235987755982988 upper=0.5235987755982988 effort=50000 velocity=50000
- joint base_link_fixed_joint: origin xyz=0 0 0.16 rpy=0 0 0 -> xyz=0.074 0 0.63 rpy=0 0 0
- joint l_gripper_fixed_joint: origin xyz=0 0.001 -0.065 rpy=-1.5707963267948961 1.570796326794896 0 -> xyz=0 -0.024941 -0.065778 rpy=3.141592653589793 1.221730955967807 -1.5707963267948968; parent l_hand -> l_hand_root
- joint l_shoulder_pitch: axis 0.0 -0.984808 -0.173648 -> 0.0 -0.970296 -0.241922; origin xyz=-0.084 0.157 0.34 rpy=0 0 0 -> xyz=-0.084 0.17 0.34 rpy=0 0 0
- joint l_wrist_fixed_joint: origin xyz=0 0.001 0 rpy=0 0 0 -> xyz=0 -0.001 0 rpy=0 0 0; parent l_hand -> l_hand_root
- joint mobile_base_l_wheel: limit (none) -> lower=-17.43583922742335 upper=17.43583922742335 effort=50000 velocity=50000; type continuous -> revolute
- joint mobile_base_r_wheel: limit (none) -> lower=-17.43583922742335 upper=17.43583922742335 effort=50000 velocity=50000; type continuous -> revolute
- joint r_gripper_fixed_joint: origin xyz=0 -0.001 -0.065 rpy=-1.5707963267948961 1.570796326794896 0 -> xyz=0 0.022941 -0.065778 rpy=0 1.221730955967806 1.5707963267948957; parent r_hand -> r_hand_root
- joint r_shoulder_pitch: axis 0.0 -0.984808 0.173648 -> 0.0 -0.970296 0.241922; origin xyz=-0.084 -0.157 0.34 rpy=0 0 0 -> xyz=-0.084 -0.17 0.34 rpy=0 0 0
- joint r_wrist_fixed_joint: parent r_hand -> r_hand_root
- joint torso_yaw: limit lower=-1.5707963267948966 upper=1.5707963267948966 effort=50000 velocity=50000 -> lower=-1.0471975511965976 upper=1.0471975511965976 effort=50000 velocity=50000
