Commit message: corrected path to meshes

File: catkin_ws/src/cer_rviz/urdf/cer.urdf (robot description, URDF)
Before this commit: robot SIM_CER_ROBOT, 58 links, 57 joints
Links:
- link chest_link: geometry collision mesh filename=package://cer_rviz/urdf/meshes/dae/sim_cer_chest.dae scale=0.001 0.001 0.001; visual mesh filename=package://cer_rviz/urdf/meshes/dae/sim_cer_chest.dae scale=0.001 0.001 0.001
- link head_link: geometry collision mesh filename=package://cer_rviz/urdf/meshes/dae/sim_cer_head.dae scale=0.001 0.001 0.001; visual mesh filename=package://cer_rviz/urdf/meshes/dae/sim_cer_head.dae scale=0.001 0.001 0.001
- link l_clavicle_link: geometry collision mesh filename=package://cer_rviz/urdf/meshes/dae/sim_cer_l_clavicle.dae scale=0.001 0.001 0.001; visual mesh filename=package://cer_rviz/urdf/meshes/dae/sim_cer_l_clavicle.dae scale=0.001 0.001 0.001
- link l_elbow_sphere_link: geometry collision mesh filename=package://cer_rviz/urdf/meshes/dae/sim_cer_l_elbow_sphere.d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 scale=0.001 0.001 0.001; visual mesh filename=package://cer_rviz/urdf/meshes/dae/sim_cer_l_elbow_sphere.d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 scale=0.001 0.001 0.001
- link l_forearm_link: geometry collision mesh filename=package://cer_rviz/urdf/meshes/dae/sim_cer_l_forearm.dae scale=0.001 0.001 0.001; visual mesh filename=package://cer_rviz/urdf/meshes/dae/sim_cer_l_forearm.dae scale=0.001 0.001 0.001
- link l_hand_paddle_distal_link: geometry collision mesh filename=package://cer_rviz/urdf/meshes/dae/sim_cer_l_hand_paddle_di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 scale=0.001 0.001 0.001; visual mesh filename=package://cer_rviz/urdf/meshes/dae/sim_cer_l_hand_paddle_di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 scale=0.001 0.001 0.001
- link l_hand_paddle_proximal_link: geometry collision mesh filename=package://cer_rviz/urdf/meshes/dae/sim_cer_l_hand_paddle_pr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 scale=0.001 0.001 0.001; visual mesh filename=package://cer_rviz/urdf/meshes/dae/sim_cer_l_hand_paddle_pr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 scale=0.001 0.001 0.001
- link l_hand_root_link: geometry collision mesh filename=package://cer_rviz/urdf/meshes/dae/sim_cer_l_hand_root.dae scale=0.001 0.001 0.001; visual mesh filename=package://cer_rviz/urdf/meshes/dae/sim_cer_l_hand_root.dae scale=0.001 0.001 0.001
- link l_hand_thumb_distal_link: geometry collision mesh filename=package://cer_rviz/urdf/meshes/dae/sim_cer_l_hand_thumb_dis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 scale=0.001 0.001 0.001; visual mesh filename=package://cer_rviz/urdf/meshes/dae/sim_cer_l_hand_thumb_dis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 scale=0.001 0.001 0.001
- link l_hand_thumb_proximal_link: geometry collision mesh filename=package://cer_rviz/urdf/meshes/dae/sim_cer_l_hand_thumb_pro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 scale=0.001 0.001 0.001; visual mesh filename=package://cer_rviz/urdf/meshes/dae/sim_cer_l_hand_thumb_pro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 scale=0.001 0.001 0.001
- link l_shoulder_link: geometry collision mesh filename=package://cer_rviz/urdf/meshes/dae/sim_cer_l_shoulder.dae scale=0.001 0.001 0.001; visual mesh filename=package://cer_rviz/urdf/meshes/dae/sim_cer_l_shoulder.dae scale=0.001 0.001 0.001
- link l_upperarm_FT_sensor_link: geometry collision mesh filename=package://cer_rviz/urdf/meshes/dae/sim_cer_l_upperarm_senso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 scale=0.001 0.001 0.001; visual mesh filename=package://cer_rviz/urdf/meshes/dae/sim_cer_l_upperarm_senso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 scale=0.001 0.001 0.001
- link l_upperarm_link: geometry collision mesh filename=package://cer_rviz/urdf/meshes/dae/sim_cer_l_upperarm.dae scale=0.001 0.001 0.001; visual mesh filename=package://cer_rviz/urdf/meshes/dae/sim_cer_l_upperarm.dae scale=0.001 0.001 0.001
- link l_wrist_cup_eq_link: geometry collision mesh filename=package://cer_rviz/urdf/meshes/dae/sim_cer_l_wrist_cup_eq.d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 scale=0.001 0.001 0.001; visual mesh filename=package://cer_rviz/urdf/meshes/dae/sim_cer_l_wrist_cup_eq.d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 scale=0.001 0.001 0.001
- link l_wrist_slider_eq_link: geometry collision mesh filename=package://cer_rviz/urdf/meshes/dae/sim_cer_l_wrist_slider.d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 scale=0.001 0.001 0.001; visual mesh filename=package://cer_rviz/urdf/meshes/dae/sim_cer_l_wrist_slider.d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 scale=0.001 0.001 0.001
- link mobile_base_body_link: geometry collision mesh filename=package://cer_rviz/urdf/meshes/dae/sim_cer_mobilebase_body.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 scale=0.001 0.001 0.001; visual mesh filename=package://cer_rviz/urdf/meshes/dae/sim_cer_mobilebase_body.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 scale=0.001 0.001 0.001
- link mobile_base_l_tyre_link: geometry collision cylinder length=0.005 radius=0.16; visual mesh filename=package://cer_rviz/urdf/meshes/dae/sim_cer_mobilebase_l_tyr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 scale=0.001 0.001 0.001
- link mobile_base_r_tyre_link: geometry collision cylinder length=0.005 radius=0.16; visual mesh filename=package://cer_rviz/urdf/meshes/dae/sim_cer_mobilebase_r_tyr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 scale=0.001 0.001 0.001
- link neck_link: geometry collision mesh filename=package://cer_rviz/urdf/meshes/dae/sim_cer_neck.dae scale=0.001 0.001 0.001; visual mesh filename=package://cer_rviz/urdf/meshes/dae/sim_cer_neck.dae scale=0.001 0.001 0.001
- link r_clavicle_link: geometry collision mesh filename=package://cer_rviz/urdf/meshes/dae/sim_cer_r_clavicle.dae scale=0.001 0.001 0.001; visual mesh filename=package://cer_rviz/urdf/meshes/dae/sim_cer_r_clavicle.dae scale=0.001 0.001 0.001
- link r_elbow_sphere_link: geometry collision mesh filename=package://cer_rviz/urdf/meshes/dae/sim_cer_r_elbow_sphere.d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 scale=0.001 0.001 0.001; visual mesh filename=package://cer_rviz/urdf/meshes/dae/sim_cer_r_elbow_sphere.d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 scale=0.001 0.001 0.001
- link r_forearm_link: geometry collision mesh filename=package://cer_rviz/urdf/meshes/dae/sim_cer_r_forearm.dae scale=0.001 0.001 0.001; visual mesh filename=package://cer_rviz/urdf/meshes/dae/sim_cer_r_forearm.dae scale=0.001 0.001 0.001
- link r_hand_paddle_distal_link: geometry collision mesh filename=package://cer_rviz/urdf/meshes/dae/sim_cer_r_hand_paddle_di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 scale=0.001 0.001 0.001; visual mesh filename=package://cer_rviz/urdf/meshes/dae/sim_cer_r_hand_paddle_di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 scale=0.001 0.001 0.001
- link r_hand_paddle_proximal_link: geometry collision mesh filename=package://cer_rviz/urdf/meshes/dae/sim_cer_r_hand_paddle_pr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 scale=0.001 0.001 0.001; visual mesh filename=package://cer_rviz/urdf/meshes/dae/sim_cer_r_hand_paddle_pr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 scale=0.001 0.001 0.001
- link r_hand_root_link: geometry collision mesh filename=package://cer_rviz/urdf/meshes/dae/sim_cer_r_hand_root.dae scale=0.001 0.001 0.001; visual mesh filename=package://cer_rviz/urdf/meshes/dae/sim_cer_r_hand_root.dae scale=0.001 0.001 0.001
- link r_hand_thumb_distal_link: geometry collision mesh filename=package://cer_rviz/urdf/meshes/dae/sim_cer_r_hand_thumb_dis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 scale=0.001 0.001 0.001; visual mesh filename=package://cer_rviz/urdf/meshes/dae/sim_cer_r_hand_thumb_dis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 scale=0.001 0.001 0.001
- link r_hand_thumb_proximal_link: geometry collision mesh filename=package://cer_rviz/urdf/meshes/dae/sim_cer_r_hand_thumb_pro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 scale=0.001 0.001 0.001; visual mesh filename=package://cer_rviz/urdf/meshes/dae/sim_cer_r_hand_thumb_pro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 scale=0.001 0.001 0.001
- link r_shoulder_link: geometry collision mesh filename=package://cer_rviz/urdf/meshes/dae/sim_cer_r_shoulder.dae scale=0.001 0.001 0.001; visual mesh filename=package://cer_rviz/urdf/meshes/dae/sim_cer_r_shoulder.dae scale=0.001 0.001 0.001
- link r_upperarm_FT_sensor_link: geometry collision mesh filename=package://cer_rviz/urdf/meshes/dae/sim_cer_r_upperarm_senso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 scale=0.001 0.001 0.001; visual mesh filename=package://cer_rviz/urdf/meshes/dae/sim_cer_r_upperarm_senso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 scale=0.001 0.001 0.001
- link r_upperarm_link: geometry collision mesh filename=package://cer_rviz/urdf/meshes/dae/sim_cer_r_upperarm.dae scale=0.001 0.001 0.001; visual mesh filename=package://cer_rviz/urdf/meshes/dae/sim_cer_r_upperarm.dae scale=0.001 0.001 0.001
- link r_wrist_cup_eq_link: geometry collision mesh filename=package://cer_rviz/urdf/meshes/dae/sim_cer_r_wrist_cup_eq.d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 scale=0.001 0.001 0.001; visual mesh filename=package://cer_rviz/urdf/meshes/dae/sim_cer_r_wrist_cup_eq.d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 scale=0.001 0.001 0.001
- link r_wrist_slider_eq_link: geometry collision mesh filename=package://cer_rviz/urdf/meshes/dae/sim_cer_r_wrist_slider.d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 scale=0.001 0.001 0.001; visual mesh filename=package://cer_rviz/urdf/meshes/dae/sim_cer_r_wrist_slider.d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 scale=0.001 0.001 0.001
- link torso_pin_eq_link: geometry collision mesh filename=package://cer_rviz/urdf/meshes/dae/sim_cer_torso_pin_eq.dae scale=0.001 0.001 0.001; visual mesh filename=package://cer_rviz/urdf/meshes/dae/sim_cer_torso_pin_eq.dae scale=0.001 0.001 0.001
- link torso_platform_link: geometry collision mesh filename=package://cer_rviz/urdf/meshes/dae/sim_cer_torso_platform.d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 scale=0.001 0.001 0.001; visual mesh filename=package://cer_rviz/urdf/meshes/dae/sim_cer_torso_platform.d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 scale=0.001 0.001 0.001
- link torso_slider_eq_link: geometry collision mesh filename=package://cer_rviz/urdf/meshes/dae/sim_cer_torso_slider_eq.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 scale=0.001 0.001 0.001; visual mesh filename=package://cer_rviz/urdf/meshes/dae/sim_cer_torso_slider_eq.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 scale=0.001 0.001 0.001

Commit message: Update catkin_ws/src/cer_rviz/urdf/cer.urdf from robots-configuration

File: catkin_ws/src/cer_rviz/urdf/cer.urdf (robot description, URDF)
Before this commit: robot SIM_CER_ROBOT, 58 links, 57 joints
Links:
- removed link mobile_base_lidar
- added link ground_link
- added link mobile_base_double_lidar
- added link mobile_base_lidar_B
- added link mobile_base_lidar_F
Joints:
- removed joint mobile_base_lidar_fixed_joint
- added joint ground_link_fixed_joint: type fixed, parent base_link, child ground_link, origin xyz=0 0 -0.2 rpy=0 0 0
- added joint mobile_base_double_lidar_fixed_joint: type fixed, parent mobile_base_body_link, child mobile_base_double_lidar, origin xyz=0.0 0 0.031 rpy=0 0 0
- added joint mobile_base_lidar_B_fixed_joint: type fixed, parent mobile_base_body_link, child mobile_base_lidar_B, origin xyz=-0.085 0 0.031 rpy=0 0 3.14
- added joint mobile_base_lidar_F_fixed_joint: type fixed, parent mobile_base_body_link, child mobile_base_lidar_F, origin xyz=0.07 0 0.031 rpy=0 0 0
