Commit message: adding cameras and depth camera to robot model

File: cer-gazebo/cer/cer.urdf (robot description, URDF)
Before this commit: robot SIM_CER_ROBOT, 48 links, 47 joints
Links:
- removed link head_asus_xtion
- removed link head_left_cam
- removed link head_right_cam
- added link asus_xtion
- added link left_camera
- added link right_camera
Joints:
- removed joint head_asus_xtion_fixed_joint
- removed joint head_left_cam_fixed_joint
- removed joint head_right_cam_fixed_joint
- added joint asus_xtion_fixed_joint: type fixed, parent head, child asus_xtion, origin xyz=0.07702051 0 0.04662 rpy=0 0 0
- added joint left_camera_fixed_joint: type fixed, parent head, child left_camera, origin xyz=0.06682051 0.0325 -0.06838 rpy=0 0 0
- added joint right_camera_fixed_joint: type fixed, parent head, child right_camera, origin xyz=0.06682051 -0.0325 -0.06838 rpy=0 0 0
- joint l_elbow: limit lower=0.0 upper=2.44346095279 effort=50000 velocity=50000 -> lower=0.0 upper=2.443460952792061 effort=50000 velocity=50000
- joint l_gripper_fixed_joint: origin xyz=0 -0.024941 -0.065778 rpy=3.14159265359 1.22173095597 -1.57079632679 -> xyz=0 -0.024941 -0.065778 rpy=3.141592653589793 1.221730955967807 -1.5707963267948968
- joint l_hand_paddle_joint: limit lower=0.0 upper=1.0471975512 effort=50000 velocity=50000 -> lower=0.0 upper=1.0471975511965976 effort=50000 velocity=50000
- joint l_hand_paddle_tip_fixed_joint: origin xyz=0 0 -0.084994 rpy=3.14159265359 1.22173095597 -1.57079632679 -> xyz=0 0 -0.084994 rpy=3.141592653589793 1.221730955967807 -1.5707963267948968
- joint l_hand_thumb_joint: limit lower=0.0 upper=1.2217304764 effort=50000 velocity=50000 -> lower=0.0 upper=1.2217304763960306 effort=50000 velocity=50000
- joint l_hand_thumb_tip_fixed_joint: origin xyz=0 -0.0513860000782 -0.0458929999125 rpy=3.14159265359 1.22173095426 -1.57079632679 -> xyz=0 -0.0513860000782 -0.0458929999125 rpy=3.141592653589793 1.2217309542643466 -1.570796326794897
- joint l_shoulder_pitch: limit lower=-0.349065850399 upper=1.74532925199 effort=50000 velocity=50000 -> lower=-0.3490658503988659 upper=1.7453292519943295 effort=50000 velocity=50000
- joint l_shoulder_roll: limit lower=-0.174532925199 upper=1.74532925199 effort=50000 velocity=50000 -> lower=-0.17453292519943295 upper=1.7453292519943295 effort=50000 velocity=50000
- joint l_shoulder_yaw: limit lower=-1.57079632679 upper=1.57079632679 effort=50000 velocity=50000 -> lower=-1.5707963267948966 upper=1.5707963267948966 effort=50000 velocity=50000
- joint l_wrist_prosupination: limit lower=-1.57079632679 upper=1.57079632679 effort=50000 velocity=50000 -> lower=-1.5707963267948966 upper=1.5707963267948966 effort=50000 velocity=50000
- joint l_wrist_tripod_pitch_eq: limit lower=-0.523598775598 upper=0.523598775598 effort=50000 velocity=50000 -> lower=-0.5235987755982988 upper=0.5235987755982988 effort=50000 velocity=50000; origin xyz=0 0.001 0 rpy=0 -1.57079632679 0 -> xyz=0 0.001 0 rpy=0 -1.5707963267948966 0
- joint l_wrist_tripod_roll_eq: limit lower=-0.523598775598 upper=0.523598775598 effort=50000 velocity=50000 -> lower=-0.5235987755982988 upper=0.5235987755982988 effort=50000 velocity=50000; origin xyz=0 0 -0.291 rpy=0 1.57079632679 0 -> xyz=0 0 -0.291 rpy=0 1.5707963267948966 0
- joint mobile_base_l_wheel: limit lower=-17.4358392274 upper=17.4358392274 effort=50000 velocity=50000 -> lower=-17.43583922742335 upper=17.43583922742335 effort=50000 velocity=50000
- joint mobile_base_r_wheel: limit lower=-17.4358392274 upper=17.4358392274 effort=50000 velocity=50000 -> lower=-17.43583922742335 upper=17.43583922742335 effort=50000 velocity=50000
- joint neck_pitch: limit lower=-0.523598775598 upper=1.3962634016 effort=50000 velocity=50000 -> lower=-0.5235987755982988 upper=1.3962634015954636 effort=50000 velocity=50000
- joint neck_yaw: limit lower=-1.3962634016 upper=1.3962634016 effort=50000 velocity=50000 -> lower=-1.3962634015954636 upper=1.3962634015954636 effort=50000 velocity=50000
- joint oriented_l_wrist_tripodbase_fixed_joint: origin xyz=0 0 0 rpy=3.14159265359 0 -1.57079632679 -> xyz=0 0 0 rpy=3.141592653589793 0 -1.5707963267948966
- joint oriented_r_wrist_tripodbase_fixed_joint: origin xyz=0 0 0 rpy=3.14159265359 0 1.57079632679 -> xyz=0 0 0 rpy=3.141592653589793 0 1.5707963267948966
- joint oriented_xbk_yrg_zup_torso_tripod_platform_fixed_joint: origin xyz=0 0 0 rpy=0 0 3.14159265359 -> xyz=0 0 0 rpy=0 0 3.141592653589793
- joint r_elbow: limit lower=0.0 upper=2.44346095279 effort=50000 velocity=50000 -> lower=0.0 upper=2.443460952792061 effort=50000 velocity=50000
- joint r_gripper_fixed_joint: origin xyz=0 0.022941 -0.065778 rpy=0 1.22173095597 1.57079632679 -> xyz=0 0.022941 -0.065778 rpy=0 1.221730955967806 1.5707963267948957
- joint r_hand_paddle_joint: limit lower=0.0 upper=1.0471975512 effort=50000 velocity=50000 -> lower=0.0 upper=1.0471975511965976 effort=50000 velocity=50000
- joint r_hand_paddle_tip_fixed_joint: origin xyz=0 0 -0.084994 rpy=0 1.22173095597 1.57079632679 -> xyz=0 0 -0.084994 rpy=0 1.221730955967806 1.5707963267948957
- joint r_hand_thumb_joint: limit lower=0.0 upper=1.2217304764 effort=50000 velocity=50000 -> lower=0.0 upper=1.2217304763960306 effort=50000 velocity=50000
- joint r_hand_thumb_tip_fixed_joint: origin xyz=0 0.051386 -0.045893 rpy=0 1.22173095597 1.57079632679 -> xyz=0 0.051386 -0.045893 rpy=0 1.221730955967806 1.5707963267948957
- joint r_shoulder_pitch: limit lower=-0.349065850399 upper=1.74532925199 effort=50000 velocity=50000 -> lower=-0.3490658503988659 upper=1.7453292519943295 effort=50000 velocity=50000
- joint r_shoulder_roll: limit lower=-0.174532925199 upper=1.74532925199 effort=50000 velocity=50000 -> lower=-0.17453292519943295 upper=1.7453292519943295 effort=50000 velocity=50000
- joint r_shoulder_yaw: limit lower=-1.57079632679 upper=1.57079632679 effort=50000 velocity=50000 -> lower=-1.5707963267948966 upper=1.5707963267948966 effort=50000 velocity=50000
- joint r_wrist_prosupination: limit lower=-1.57079632679 upper=1.57079632679 effort=50000 velocity=50000 -> lower=-1.5707963267948966 upper=1.5707963267948966 effort=50000 velocity=50000
- joint r_wrist_tripod_pitch_eq: limit lower=-0.523598775598 upper=0.523598775598 effort=50000 velocity=50000 -> lower=-0.5235987755982988 upper=0.5235987755982988 effort=50000 velocity=50000; origin xyz=0.001 0 0 rpy=3.14159265359 0 1.57079632679 -> xyz=0.001 0 0 rpy=3.141592653589793 0 1.5707963267948966
- joint r_wrist_tripod_roll_eq: limit lower=-0.523598775598 upper=0.523598775598 effort=50000 velocity=50000 -> lower=-0.5235987755982988 upper=0.5235987755982988 effort=50000 velocity=50000; origin xyz=0 0 -0.291 rpy=3.14159265359 0 1.57079632679 -> xyz=0 0 -0.291 rpy=3.141592653589793 0 1.5707963267948966
- joint torso_tripod_pitch_eq: limit lower=-0.523598775598 upper=0.523598775598 effort=50000 velocity=50000 -> lower=-0.5235987755982988 upper=0.5235987755982988 effort=50000 velocity=50000; origin xyz=0 0 0 rpy=3.14159265359 0 0 -> xyz=0 0 0 rpy=3.141592653589793 0 0
- joint torso_tripod_roll_eq: limit lower=-0.523598775598 upper=0.523598775598 effort=50000 velocity=50000 -> lower=-0.5235987755982988 upper=0.5235987755982988 effort=50000 velocity=50000; origin xyz=0 0 0.399 rpy=3.14159265359 0 0 -> xyz=0 0 0.399 rpy=3.141592653589793 0 0
- joint torso_yaw: limit lower=-1.0471975512 upper=1.0471975512 effort=50000 velocity=50000 -> lower=-1.0471975511965976 upper=1.0471975511965976 effort=50000 velocity=50000
