Commit message: minor fix in joint name and range

File: cer-gazebo/cer2/cer.urdf (robot description, URDF)
Before this commit: robot SIM_CER_ROBOT, 55 links, 54 joints
Joints:
- removed joint l_wrist_prosupination_joint
- removed joint r_wrist_prosupination_joint
- added joint l_wrist_pronosupination_joint: type revolute, parent l_elbow_sphere_link, child l_forearm_link, origin xyz=0 0 -0.071 rpy=0 0 0, axis 0.0 0.0 1.0, limit lower=-1.57079632679 upper=1.57079632679 effort=10.0 velocity=3.14
- added joint r_wrist_pronosupination_joint: type revolute, parent r_elbow_sphere_link, child r_forearm_link, origin xyz=0 0 -0.071 rpy=0 0 0, axis 0.0 0.0 -1.0, limit lower=-1.57079632679 upper=1.57079632679 effort=10.0 velocity=3.14
- joint l_elbow_joint: limit lower=0.0 upper=1.76278254451 effort=20.0 velocity=3.14 -> lower=0.0 upper=1.74532925199 effort=20.0 velocity=3.14
- joint r_elbow_joint: limit lower=0.0 upper=1.76278254451 effort=20.0 velocity=3.14 -> lower=0.0 upper=1.74532925199 effort=20.0 velocity=3.14
- joint torso_pitch_eq_joint: limit lower=-0.523598775598 upper=0.523598775598 effort=30.0 velocity=3.14 -> lower=-0.523598775598 upper=0.523598775598 effort=50.0 velocity=3.14
- joint torso_roll_eq_joint: limit lower=-0.523598775598 upper=0.523598775598 effort=30.0 velocity=3.14 -> lower=-0.523598775598 upper=0.523598775598 effort=50.0 velocity=3.14

Commit message: Use relative path to find meshes file

File: cer-gazebo/cer2/cer.urdf (robot description, URDF)
Before this commit: robot SIM_CER_ROBOT, 55 links, 54 joints
Links:
- link chest_link: geometry collision mesh filename=package://cer_rviz/../../../cer-gazebo/cer2/meshes/dae/sim_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 scale=0.001 0.001 0.001; visual mesh filename=package://cer_rviz/../../../cer-gazebo/cer2/meshes/dae/sim_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 scale=0.001 0.001 0.001
- link head_link: geometry collision mesh filename=package://cer_rviz/../../../cer-gazebo/cer2/meshes/dae/sim_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 scale=0.001 0.001 0.001; visual mesh filename=package://cer_rviz/../../../cer-gazebo/cer2/meshes/dae/sim_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 scale=0.001 0.001 0.001
- link l_clavicle_link: geometry collision mesh filename=package://cer_rviz/../../../cer-gazebo/cer2/meshes/dae/sim_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 scale=0.001 0.001 0.001; visual mesh filename=package://cer_rviz/../../../cer-gazebo/cer2/meshes/dae/sim_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 scale=0.001 0.001 0.001
- link l_elbow_sphere_link: geometry collision mesh filename=package://cer_rviz/../../../cer-gazebo/cer2/meshes/dae/sim_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 scale=0.001 0.001 0.001; visual mesh filename=package://cer_rviz/../../../cer-gazebo/cer2/meshes/dae/sim_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 scale=0.001 0.001 0.001
- link l_forearm_link: geometry collision mesh filename=package://cer_rviz/../../../cer-gazebo/cer2/meshes/dae/sim_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 scale=0.001 0.001 0.001; visual mesh filename=package://cer_rviz/../../../cer-gazebo/cer2/meshes/dae/sim_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 scale=0.001 0.001 0.001
- link l_hand_paddle_distal_link: geometry collision mesh filename=package://cer_rviz/../../../cer-gazebo/cer2/meshes/dae/sim_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 scale=0.001 0.001 0.001; visual mesh filename=package://cer_rviz/../../../cer-gazebo/cer2/meshes/dae/sim_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 scale=0.001 0.001 0.001
- link l_hand_paddle_proximal_link: geometry collision mesh filename=package://cer_rviz/../../../cer-gazebo/cer2/meshes/dae/sim_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 scale=0.001 0.001 0.001; visual mesh filename=package://cer_rviz/../../../cer-gazebo/cer2/meshes/dae/sim_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 scale=0.001 0.001 0.001
- link l_hand_root_link: geometry collision mesh filename=package://cer_rviz/../../../cer-gazebo/cer2/meshes/dae/sim_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 scale=0.001 0.001 0.001; visual mesh filename=package://cer_rviz/../../../cer-gazebo/cer2/meshes/dae/sim_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 scale=0.001 0.001 0.001
- link l_hand_thumb_distal_link: geometry collision mesh filename=package://cer_rviz/../../../cer-gazebo/cer2/meshes/dae/sim_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 scale=0.001 0.001 0.001; visual mesh filename=package://cer_rviz/../../../cer-gazebo/cer2/meshes/dae/sim_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 scale=0.001 0.001 0.001
- link l_hand_thumb_proximal_link: geometry collision mesh filename=package://cer_rviz/../../../cer-gazebo/cer2/meshes/dae/sim_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 scale=0.001 0.001 0.001; visual mesh filename=package://cer_rviz/../../../cer-gazebo/cer2/meshes/dae/sim_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 scale=0.001 0.001 0.001
- link l_shoulder_link: geometry collision mesh filename=package://cer_rviz/../../../cer-gazebo/cer2/meshes/dae/sim_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 scale=0.001 0.001 0.001; visual mesh filename=package://cer_rviz/../../../cer-gazebo/cer2/meshes/dae/sim_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 scale=0.001 0.001 0.001
- link l_upperarm_FT_sensor_link: geometry collision mesh filename=package://cer_rviz/../../../cer-gazebo/cer2/meshes/dae/sim_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 scale=0.001 0.001 0.001; visual mesh filename=package://cer_rviz/../../../cer-gazebo/cer2/meshes/dae/sim_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 scale=0.001 0.001 0.001
- link l_upperarm_link: geometry collision mesh filename=package://cer_rviz/../../../cer-gazebo/cer2/meshes/dae/sim_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 scale=0.001 0.001 0.001; visual mesh filename=package://cer_rviz/../../../cer-gazebo/cer2/meshes/dae/sim_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 scale=0.001 0.001 0.001
- link l_wrist_cup_eq_link: geometry collision mesh filename=package://cer_rviz/../../../cer-gazebo/cer2/meshes/dae/sim_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 scale=0.001 0.001 0.001; visual mesh filename=package://cer_rviz/../../../cer-gazebo/cer2/meshes/dae/sim_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 scale=0.001 0.001 0.001
- link l_wrist_slider_eq_link: geometry collision mesh filename=package://cer_rviz/../../../cer-gazebo/cer2/meshes/dae/sim_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 scale=0.001 0.001 0.001; visual mesh filename=package://cer_rviz/../../../cer-gazebo/cer2/meshes/dae/sim_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 scale=0.001 0.001 0.001
- link mobile_base_body_link: geometry collision mesh filename=package://cer_rviz/../../../cer-gazebo/cer2/meshes/dae/sim_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 scale=0.001 0.001 0.001; visual mesh filename=package://cer_rviz/../../../cer-gazebo/cer2/meshes/dae/sim_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 scale=0.001 0.001 0.001
- link mobile_base_l_tyre_link: geometry collision cylinder length=0.06 radius=0.16; visual mesh filename=package://cer_rviz/../../../cer-gazebo/cer2/meshes/dae/sim_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 scale=0.001 0.001 0.001
- link mobile_base_r_tyre_link: geometry collision cylinder length=0.06 radius=0.16; visual mesh filename=package://cer_rviz/../../../cer-gazebo/cer2/meshes/dae/sim_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 scale=0.001 0.001 0.001
- link neck_link: geometry collision mesh filename=package://cer_rviz/../../../cer-gazebo/cer2/meshes/dae/sim_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 scale=0.001 0.001 0.001; visual mesh filename=package://cer_rviz/../../../cer-gazebo/cer2/meshes/dae/sim_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 scale=0.001 0.001 0.001
- link r_clavicle_link: geometry collision mesh filename=package://cer_rviz/../../../cer-gazebo/cer2/meshes/dae/sim_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 scale=0.001 0.001 0.001; visual mesh filename=package://cer_rviz/../../../cer-gazebo/cer2/meshes/dae/sim_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 scale=0.001 0.001 0.001
- link r_elbow_sphere_link: geometry collision mesh filename=package://cer_rviz/../../../cer-gazebo/cer2/meshes/dae/sim_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 scale=0.001 0.001 0.001; visual mesh filename=package://cer_rviz/../../../cer-gazebo/cer2/meshes/dae/sim_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 scale=0.001 0.001 0.001
- link r_forearm_link: geometry collision mesh filename=package://cer_rviz/../../../cer-gazebo/cer2/meshes/dae/sim_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 scale=0.001 0.001 0.001; visual mesh filename=package://cer_rviz/../../../cer-gazebo/cer2/meshes/dae/sim_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 scale=0.001 0.001 0.001
- link r_hand_paddle_distal_link: geometry collision mesh filename=package://cer_rviz/../../../cer-gazebo/cer2/meshes/dae/sim_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 scale=0.001 0.001 0.001; visual mesh filename=package://cer_rviz/../../../cer-gazebo/cer2/meshes/dae/sim_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 scale=0.001 0.001 0.001
- link r_hand_paddle_proximal_link: geometry collision mesh filename=package://cer_rviz/../../../cer-gazebo/cer2/meshes/dae/sim_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 scale=0.001 0.001 0.001; visual mesh filename=package://cer_rviz/../../../cer-gazebo/cer2/meshes/dae/sim_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 scale=0.001 0.001 0.001
- link r_hand_root_link: geometry collision mesh filename=package://cer_rviz/../../../cer-gazebo/cer2/meshes/dae/sim_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 scale=0.001 0.001 0.001; visual mesh filename=package://cer_rviz/../../../cer-gazebo/cer2/meshes/dae/sim_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 scale=0.001 0.001 0.001
- link r_hand_thumb_distal_link: geometry collision mesh filename=package://cer_rviz/../../../cer-gazebo/cer2/meshes/dae/sim_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 scale=0.001 0.001 0.001; visual mesh filename=package://cer_rviz/../../../cer-gazebo/cer2/meshes/dae/sim_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 scale=0.001 0.001 0.001
- link r_hand_thumb_proximal_link: geometry collision mesh filename=package://cer_rviz/../../../cer-gazebo/cer2/meshes/dae/sim_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 scale=0.001 0.001 0.001; visual mesh filename=package://cer_rviz/../../../cer-gazebo/cer2/meshes/dae/sim_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 scale=0.001 0.001 0.001
- link r_shoulder_link: geometry collision mesh filename=package://cer_rviz/../../../cer-gazebo/cer2/meshes/dae/sim_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 scale=0.001 0.001 0.001; visual mesh filename=package://cer_rviz/../../../cer-gazebo/cer2/meshes/dae/sim_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 scale=0.001 0.001 0.001
- link r_upperarm_FT_sensor_link: geometry collision mesh filename=package://cer_rviz/../../../cer-gazebo/cer2/meshes/dae/sim_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 scale=0.001 0.001 0.001; visual mesh filename=package://cer_rviz/../../../cer-gazebo/cer2/meshes/dae/sim_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 scale=0.001 0.001 0.001
- link r_upperarm_link: geometry collision mesh filename=package://cer_rviz/../../../cer-gazebo/cer2/meshes/dae/sim_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 scale=0.001 0.001 0.001; visual mesh filename=package://cer_rviz/../../../cer-gazebo/cer2/meshes/dae/sim_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 scale=0.001 0.001 0.001
- link r_wrist_cup_eq_link: geometry collision mesh filename=package://cer_rviz/../../../cer-gazebo/cer2/meshes/dae/sim_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 scale=0.001 0.001 0.001; visual mesh filename=package://cer_rviz/../../../cer-gazebo/cer2/meshes/dae/sim_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 scale=0.001 0.001 0.001
- link r_wrist_slider_eq_link: geometry collision mesh filename=package://cer_rviz/../../../cer-gazebo/cer2/meshes/dae/sim_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 scale=0.001 0.001 0.001; visual mesh filename=package://cer_rviz/../../../cer-gazebo/cer2/meshes/dae/sim_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 scale=0.001 0.001 0.001
- link torso_pin_eq_link: geometry collision mesh filename=package://cer_rviz/../../../cer-gazebo/cer2/meshes/dae/sim_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 scale=0.001 0.001 0.001; visual mesh filename=package://cer_rviz/../../../cer-gazebo/cer2/meshes/dae/sim_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 scale=0.001 0.001 0.001
- link torso_platform_link: geometry collision mesh filename=package://cer_rviz/../../../cer-gazebo/cer2/meshes/dae/sim_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 scale=0.001 0.001 0.001; visual mesh filename=package://cer_rviz/../../../cer-gazebo/cer2/meshes/dae/sim_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 scale=0.001 0.001 0.001
- link torso_slider_eq_link: geometry collision mesh filename=package://cer_rviz/../../../cer-gazebo/cer2/meshes/dae/sim_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 scale=0.001 0.001 0.001; visual mesh filename=package://cer_rviz/../../../cer-gazebo/cer2/meshes/dae/sim_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 scale=0.001 0.001 0.001
