Commit message: Little correction on cer.urdf
The "mesh" tags and the "yarpConfigurationFile" where pointing to
"cer_rviz" folder instead of "cer_rviz2".

File: colcon_ws/src/cer_rviz2/urdf/cer.urdf (robot description, URDF)
Before this commit: robot SIM_CER_ROBOT, 61 links, 60 joints
Links:
- link chest_link: geometry collision mesh filename=package://cer_rviz2/urdf/meshes/dae/sim_cer_chest.dae scale=0.001 0.001 0.001; visual mesh filename=package://cer_rviz2/urdf/meshes/dae/sim_cer_chest.dae scale=0.001 0.001 0.001
- link head_link: geometry collision mesh filename=package://cer_rviz2/urdf/meshes/dae/sim_cer_head.dae scale=0.001 0.001 0.001; visual mesh filename=package://cer_rviz2/urdf/meshes/dae/sim_cer_head.dae scale=0.001 0.001 0.001
- link l_clavicle_link: geometry collision mesh filename=package://cer_rviz2/urdf/meshes/dae/sim_cer_l_clavicle.dae scale=0.001 0.001 0.001; visual mesh filename=package://cer_rviz2/urdf/meshes/dae/sim_cer_l_clavicle.dae scale=0.001 0.001 0.001
- link l_elbow_sphere_link: geometry collision mesh filename=package://cer_rviz2/urdf/meshes/dae/sim_cer_l_elbow_sphere.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 scale=0.001 0.001 0.001; visual mesh filename=package://cer_rviz2/urdf/meshes/dae/sim_cer_l_elbow_sphere.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 scale=0.001 0.001 0.001
- link l_forearm_link: geometry collision mesh filename=package://cer_rviz2/urdf/meshes/dae/sim_cer_l_forearm.dae scale=0.001 0.001 0.001; visual mesh filename=package://cer_rviz2/urdf/meshes/dae/sim_cer_l_forearm.dae scale=0.001 0.001 0.001
- link l_hand_paddle_distal_link: geometry collision mesh filename=package://cer_rviz2/urdf/meshes/dae/sim_cer_l_hand_paddle_d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 scale=0.001 0.001 0.001; visual mesh filename=package://cer_rviz2/urdf/meshes/dae/sim_cer_l_hand_paddle_d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 scale=0.001 0.001 0.001
- link l_hand_paddle_proximal_link: geometry collision mesh filename=package://cer_rviz2/urdf/meshes/dae/sim_cer_l_hand_paddle_p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 scale=0.001 0.001 0.001; visual mesh filename=package://cer_rviz2/urdf/meshes/dae/sim_cer_l_hand_paddle_p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 scale=0.001 0.001 0.001
- link l_hand_root_link: geometry collision mesh filename=package://cer_rviz2/urdf/meshes/dae/sim_cer_l_hand_root.dae scale=0.001 0.001 0.001; visual mesh filename=package://cer_rviz2/urdf/meshes/dae/sim_cer_l_hand_root.dae scale=0.001 0.001 0.001
- link l_hand_thumb_distal_link: geometry collision mesh filename=package://cer_rviz2/urdf/meshes/dae/sim_cer_l_hand_thumb_di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 scale=0.001 0.001 0.001; visual mesh filename=package://cer_rviz2/urdf/meshes/dae/sim_cer_l_hand_thumb_di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 scale=0.001 0.001 0.001
- link l_hand_thumb_proximal_link: geometry collision mesh filename=package://cer_rviz2/urdf/meshes/dae/sim_cer_l_hand_thumb_pr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 scale=0.001 0.001 0.001; visual mesh filename=package://cer_rviz2/urdf/meshes/dae/sim_cer_l_hand_thumb_pr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 scale=0.001 0.001 0.001
- link l_shoulder_link: geometry collision mesh filename=package://cer_rviz2/urdf/meshes/dae/sim_cer_l_shoulder.dae scale=0.001 0.001 0.001; visual mesh filename=package://cer_rviz2/urdf/meshes/dae/sim_cer_l_shoulder.dae scale=0.001 0.001 0.001
- link l_upperarm_FT_sensor_link: geometry collision mesh filename=package://cer_rviz2/urdf/meshes/dae/sim_cer_l_upperarm_sens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 scale=0.001 0.001 0.001; visual mesh filename=package://cer_rviz2/urdf/meshes/dae/sim_cer_l_upperarm_sens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 scale=0.001 0.001 0.001
- link l_upperarm_link: geometry collision mesh filename=package://cer_rviz2/urdf/meshes/dae/sim_cer_l_upperarm.dae scale=0.001 0.001 0.001; visual mesh filename=package://cer_rviz2/urdf/meshes/dae/sim_cer_l_upperarm.dae scale=0.001 0.001 0.001
- link l_wrist_cup_eq_link: geometry collision mesh filename=package://cer_rviz2/urdf/meshes/dae/sim_cer_l_wrist_cup_eq.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 scale=0.001 0.001 0.001; visual mesh filename=package://cer_rviz2/urdf/meshes/dae/sim_cer_l_wrist_cup_eq.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 scale=0.001 0.001 0.001
- link l_wrist_slider_eq_link: geometry collision mesh filename=package://cer_rviz2/urdf/meshes/dae/sim_cer_l_wrist_slider.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 scale=0.001 0.001 0.001; visual mesh filename=package://cer_rviz2/urdf/meshes/dae/sim_cer_l_wrist_slider.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 scale=0.001 0.001 0.001
- link mobile_base_body_link: geometry collision mesh filename=package://cer_rviz2/urdf/meshes/dae/sim_cer_mobilebase_body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 scale=0.001 0.001 0.001; visual mesh filename=package://cer_rviz2/urdf/meshes/dae/sim_cer_mobilebase_body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 scale=0.001 0.001 0.001
- link mobile_base_l_tyre_link: geometry collision cylinder length=0.005 radius=0.16; visual mesh filename=package://cer_rviz2/urdf/meshes/dae/sim_cer_mobilebase_l_ty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 scale=0.001 0.001 0.001
- link mobile_base_r_tyre_link: geometry collision cylinder length=0.005 radius=0.16; visual mesh filename=package://cer_rviz2/urdf/meshes/dae/sim_cer_mobilebase_r_ty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 scale=0.001 0.001 0.001
- link neck_link: geometry collision mesh filename=package://cer_rviz2/urdf/meshes/dae/sim_cer_neck.dae scale=0.001 0.001 0.001; visual mesh filename=package://cer_rviz2/urdf/meshes/dae/sim_cer_neck.dae scale=0.001 0.001 0.001
- link r_clavicle_link: geometry collision mesh filename=package://cer_rviz2/urdf/meshes/dae/sim_cer_r_clavicle.dae scale=0.001 0.001 0.001; visual mesh filename=package://cer_rviz2/urdf/meshes/dae/sim_cer_r_clavicle.dae scale=0.001 0.001 0.001
- link r_elbow_sphere_link: geometry collision mesh filename=package://cer_rviz2/urdf/meshes/dae/sim_cer_r_elbow_sphere.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 scale=0.001 0.001 0.001; visual mesh filename=package://cer_rviz2/urdf/meshes/dae/sim_cer_r_elbow_sphere.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 scale=0.001 0.001 0.001
- link r_forearm_link: geometry collision mesh filename=package://cer_rviz2/urdf/meshes/dae/sim_cer_r_forearm.dae scale=0.001 0.001 0.001; visual mesh filename=package://cer_rviz2/urdf/meshes/dae/sim_cer_r_forearm.dae scale=0.001 0.001 0.001
- link r_hand_paddle_distal_link: geometry collision mesh filename=package://cer_rviz2/urdf/meshes/dae/sim_cer_r_hand_paddle_d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 scale=0.001 0.001 0.001; visual mesh filename=package://cer_rviz2/urdf/meshes/dae/sim_cer_r_hand_paddle_d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 scale=0.001 0.001 0.001
- link r_hand_paddle_proximal_link: geometry collision mesh filename=package://cer_rviz2/urdf/meshes/dae/sim_cer_r_hand_paddle_p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 scale=0.001 0.001 0.001; visual mesh filename=package://cer_rviz2/urdf/meshes/dae/sim_cer_r_hand_paddle_p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 scale=0.001 0.001 0.001
- link r_hand_root_link: geometry collision mesh filename=package://cer_rviz2/urdf/meshes/dae/sim_cer_r_hand_root.dae scale=0.001 0.001 0.001; visual mesh filename=package://cer_rviz2/urdf/meshes/dae/sim_cer_r_hand_root.dae scale=0.001 0.001 0.001
- link r_hand_thumb_distal_link: geometry collision mesh filename=package://cer_rviz2/urdf/meshes/dae/sim_cer_r_hand_thumb_di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 scale=0.001 0.001 0.001; visual mesh filename=package://cer_rviz2/urdf/meshes/dae/sim_cer_r_hand_thumb_di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 scale=0.001 0.001 0.001
- link r_hand_thumb_proximal_link: geometry collision mesh filename=package://cer_rviz2/urdf/meshes/dae/sim_cer_r_hand_thumb_pr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 scale=0.001 0.001 0.001; visual mesh filename=package://cer_rviz2/urdf/meshes/dae/sim_cer_r_hand_thumb_pr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 scale=0.001 0.001 0.001
- link r_shoulder_link: geometry collision mesh filename=package://cer_rviz2/urdf/meshes/dae/sim_cer_r_shoulder.dae scale=0.001 0.001 0.001; visual mesh filename=package://cer_rviz2/urdf/meshes/dae/sim_cer_r_shoulder.dae scale=0.001 0.001 0.001
- link r_upperarm_FT_sensor_link: geometry collision mesh filename=package://cer_rviz2/urdf/meshes/dae/sim_cer_r_upperarm_sens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 scale=0.001 0.001 0.001; visual mesh filename=package://cer_rviz2/urdf/meshes/dae/sim_cer_r_upperarm_sens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 scale=0.001 0.001 0.001
- link r_upperarm_link: geometry collision mesh filename=package://cer_rviz2/urdf/meshes/dae/sim_cer_r_upperarm.dae scale=0.001 0.001 0.001; visual mesh filename=package://cer_rviz2/urdf/meshes/dae/sim_cer_r_upperarm.dae scale=0.001 0.001 0.001
- link r_wrist_cup_eq_link: geometry collision mesh filename=package://cer_rviz2/urdf/meshes/dae/sim_cer_r_wrist_cup_eq.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 scale=0.001 0.001 0.001; visual mesh filename=package://cer_rviz2/urdf/meshes/dae/sim_cer_r_wrist_cup_eq.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 scale=0.001 0.001 0.001
- link r_wrist_slider_eq_link: geometry collision mesh filename=package://cer_rviz2/urdf/meshes/dae/sim_cer_r_wrist_slider.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 scale=0.001 0.001 0.001; visual mesh filename=package://cer_rviz2/urdf/meshes/dae/sim_cer_r_wrist_slider.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 scale=0.001 0.001 0.001
- link torso_pin_eq_link: geometry collision mesh filename=package://cer_rviz2/urdf/meshes/dae/sim_cer_torso_pin_eq.dae scale=0.001 0.001 0.001; visual mesh filename=package://cer_rviz2/urdf/meshes/dae/sim_cer_torso_pin_eq.dae scale=0.001 0.001 0.001
- link torso_platform_link: geometry collision mesh filename=package://cer_rviz2/urdf/meshes/dae/sim_cer_torso_platform.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 scale=0.001 0.001 0.001; visual mesh filename=package://cer_rviz2/urdf/meshes/dae/sim_cer_torso_platform.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 scale=0.001 0.001 0.001
- link torso_slider_eq_link: geometry collision mesh filename=package://cer_rviz2/urdf/meshes/dae/sim_cer_torso_slider_eq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 scale=0.001 0.001 0.001; visual mesh filename=package://cer_rviz2/urdf/meshes/dae/sim_cer_torso_slider_eq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 scale=0.001 0.001 0.001
